File: hardware/scratch/BusPirate-ng.v4.0.sch (EAGLE design)
At the start: 130 parts, among them CON1 CON-USB-F-MICRO-B, IC10 74LVC1G07DBV, IC11 IC_BUFF_SN74LVC1T45DBV, IC12 74LVC1G07DBV, IC13 IC_BUFF_SN74LVC1T45DBV, IC14 74LVC1G07DBV, IC15 IC_BUFF_SN74LVC1T45DBV, IC16 74LVC1G07DBV, IC17 IC_BUFF_SN74LVC1T45DBV, IC2 IC_MEM_23LC1024, IC3 IC_MEM_23LC1024, IC4 IC_74AC573, IC5 IC_BL1551, IC6 IC_BL1551, IC7 74HCT4066PW, IC8 74LVC1G07DBV, IC9 IC_BUFF_SN74LVC1T45DBV, J1 CON_HEADER_1X04, J2 CON_HEADER_1X03-PTH, J3 CON_HEADER_2X02-PTH, J4 CON_HEADER_1X10-RIGHT_ANGLED_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, J5 CON_HEADER_1X10-RIGHT_ANGLED_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, U1 IC_FPGA_ICE40HX4K, U2 IC_UC_STM32F103ZX, U3 IC_MEM_AT45DB041D

Commit message: move: UART_TX and UART_RX from PA9/PA10 USART1(0) to PA6/PA7 USART1(1) VREGEN from PB6 to PE1 LD1 to PD2 USBLED to PD3 V50PU from PB4 to PG0 V33PU from PB5 to PG1 USB_DET from PA15 to PF11 VEXTPU from PC6 to PF15 remove connection of Latch's IO_OE from MCU
Parts:
- removed J4: CON_HEADER_1X10-RIGHT_ANGLED_PTH_SHROUDED, dp_devices.v6:CON_HEADER_1X10-RIGHT_ANGLED_PTH_SHROUDED
- removed R15: 100R, dp_devices.v6:RESISTOR-0603
- removed RN2: 100R, dp_devices:RNETWORK
Connections:
- removed net IO_AUX0: J4.6, R15.2
- removed net IO_CLK: J4.9, RN2B.1
- removed net IO_CS: J4.7, RN2D.1
- removed net IO_MISO: J4.8, RN2C.1
- removed net IO_MOSI: J4.10, RN2A.1
- new net N$28: U2U.PA0/WKUP/USART2_CTS('0')/ADC123_IN0/TIM2_CH1_ETR/TIM5_CH1/TIM8_ETR
- new net N$29: U2U.PA2/USART2_TX('0')/TIM5_CH3/ADC123_IN2/TIM2_CH3('00'OR'01)
- new net N$30: U2U.PA3/USART2_RX('0')/TIM5_CH4/ADC123_IN3/TIM2_CH4('00'OR'01')
- new net N$31: U2U.PG2/FT/FSMC_A12
- net AUX0: no longer R15.1
- net BPIO_CLOCK: now also RN4B.1
- net BPIO_CS: now also RN4D.1
- net BPIO_MISO: now also RN4C.1
- net BPIO_MOSI: now also RN4A.1
- net CLOCK: no longer RN2B.2, RN4B.1
- net CS: no longer RN2D.2, RN4D.1
- net GND: no longer J4.1
- net IO_ADC/DAC: no longer J4.5
- net IO_OE: no longer U2U.TIM8_CH2/TIM3_CH2('11')/FT/PC7
- net LD1: now also U2U.PD2/FT/TIM3_ETR/UART5_RX; no longer U2U.TIM8_CH3/TIM3_CH3('11')/FT/PC8
- net MISO: no longer RN2C.2, RN4C.1
- net MOSI: no longer RN2A.2, RN4A.1
- net N$10: now also U2U.PA1/USART2_RTS('0')/ADC123_IN1/TIM5_CH2/TIM2_CH2('00'); no longer U2U.PG0/FT/FSMC_A10
- net SWV33: no longer J4.3
- net SWV50: no longer J4.2
- net UART_RX: now also U2U.I2C1_SDA('0')/FSMC_NADV/TIM4_CH2('0')/USART1_RX('1')/FT/PB7; no longer U2U.PA10/FT/USART1_RX('0')/TIM1_CH3('00'OR'01')
- net UART_TX: now also U2U.I2C1_SCL('0')/TIM4_CH1('0')/USART1_TX('1')/FT/PB6; no longer U2U.PA9/FT/USART1_TX('0')/TIM1_CH2('00'OR'01')
- net USBLED: now also U2U.PD3/FT/FSMC_CLK/USART2_CTS(1); no longer U2U.TIM8_CH4/TIM3_CH4('11')/FT/PC9
- net USB_DET: now also U2U.FSMC_NIOS16/FT/PF11; no longer U2U.PA15/FT/JTDI/SPI3_NSS('0')/TIM2_CH1_ETR('11')/SPI1_NSS('1')
- net V33PU: now also U2U.PG1/FT/FSMC_A11; no longer U2U.I2C1_SMBA/SPI3_MOSI('0')/TIM3_CH2('10')/SPI1_MOSI('1')/PB5
- net V50PU: now also U2U.PG0/FT/FSMC_A10; no longer U2U.SPI3_MISO('0')/TIM3_CH1('10')/SPI1_MISO('1')/NJTRST/FT/PB4
- net VEXTERN: no longer J4.4
- net VEXTPU: now also U2U.FSMC_A9/FT/PF15; no longer U2U.TIM8_CH1/TIM3_CH1('11')/FT/PC6
- net VREGEN: now also U2U.PE1/FT/FSMC_NBL1; no longer U2U.I2C1_SCL('0')/TIM4_CH1('0')/USART1_TX('1')/FT/PB6
Other:
- note removed: "FPGA Unconnected"
- moved on the sheet: C53, C54, J5, R40

Commit message: moved SRAM_CS from PB3 to PA15 reconnect BPIO_MOSI, BPIO_CLOCK, BPIO_MISO, BPIO_CS, BPIO_AUX to latch's data pins, these we're accidentally disconnected on the last update removed connection of AUX0 from latch to MCU, latch's AUX0 is now BPIO_AUX moved flash's SPI pins from SPI1(0) namely pins PA5, PA6 and PA7 to SPI1(1) pins PB3, PB4 and PB5 wire MS0 (switch) to PF12 continue routing
Connections:
- removed net +3V3: U3.!RST, U3.!WP
- removed net AUX0: IC4IC.4D, U2U.ADC12_IN8/TIM3_CH3('00'OR'10')/TIM8_CH2N/TIM1_CH2N('01')/PB0
- removed net CLOCK: IC4IC.7D
- removed net CS: IC4IC.5D
- removed net MISO: IC4IC.6D
- removed net MOSI: IC4IC.8D
- new net N$32: U2U.TIM4_CH3('0')/I2C1_SCL('1')/FT/PB8
- new net N$33: U2U.TIM4_CH4('0')/I2C1_SDA('1')/FT/PB9
- new net N$34: U2U.PA4/SPI1_NSS('0')/USART2_CK('0')/ADC12_IN4
- new net N$35: U2U.ADC12_IN15/PC5
- new net N$36: U2U.ADC3_IN4/PF6
- new net N$37: U2U.ADC3_IN5/PF7
- new net N$38: U2U.ADC3_IN6/PF8
- new net N$39: U2U.ADC_IN7/PF9
- new net N$40: U2U.ADC_IN8/PF10
- new net N$44: U2U.ADC12_IN8/TIM3_CH3('00'OR'10')/TIM8_CH2N/TIM1_CH2N('01')/PB0
- net 3V3: now also U3.!RST, U3.!WP
- net BPIO_AUX: now also IC4IC.4D
- net BPIO_CLOCK: now also IC4IC.7D
- net BPIO_CS: now also IC4IC.5D
- net BPIO_MISO: now also IC4IC.6D
- net BPIO_MOSI: now also IC4IC.8D
- net FLASH_MISO: now also U2U.SPI3_MISO('0')/TIM3_CH1('10')/SPI1_MISO('1')/NJTRST/FT/PB4; no longer U2U.PA6/SPI1_MISO('0')/TIM8_BKIN/ADC12_IN6/TIM3_CH1('00')/TIM1_BKIN('01')
- net FLASH_MOSI: now also U2U.I2C1_SMBA/SPI3_MOSI('0')/TIM3_CH2('10')/SPI1_MOSI('1')/PB5; no longer U2U.PA7/SPI1_MOSI('0')/TIM8_CH1N/ADC12_IN7/TIM3_CH2('00')/TIM1_CH1N('01')
- net FLASH_SCK: now also U2U.SPI3_SCK('0')/TIM2_CH2('01')/SPI1_SCK('1')/JTDO/FT//PB3; no longer U2U.PA5/SPI1_SCK('0')/ADC12_IN5
- net MS0: now also U2U.FSMC_A6/FT/PF12
- net SRAM_CS: now also U2U.PA15/FT/JTDI/SPI3_NSS('0')/TIM2_CH1_ETR('11')/SPI1_NSS('1'); no longer U2U.SPI3_SCK('0')/TIM2_CH2('01')/SPI1_SCK('1')/JTDO/FT//PB3

Commit message: move ADC5 from PC0 to PA3 move ADC4 from PC2 to PC4 move ADC3 from PC1 to PC5 move AD6 to PC4 move latch's IO_OE from FPGA pin IOT_206 to IOT_177 remove connection of logic analyzer's 2 SRAM CS from MCU and wire each CS to FPGA, SRAM_CS1 to FPGA's IOT_222 and SRAM_CS2 to IOT_206 move MCU to FPGA interrupt from BANK2 to BANK0, interrupt pins are on GBIN0 and GBIN1 wired interrupt pins MCU_INT0 and MCU_INT1 to PC11 and PC10 respectively
Connections:
- removed net N$23: U1BANK0.IOT_177
- removed net N$24: U1BANK0.GBIN0/IOT_198
- removed net N$25: U1BANK0.GBIN1/IOT_197
- removed net SRAM_CS: IC2IC.!CS, IC3IC.!CS, U1BANK0.IOT_222, U2U.PA15/FT/JTDI/SPI3_NSS('0')/TIM2_CH1_ETR('11')/SPI1_NSS('1')
- new net N$41: U2U.TIM8_CH4/TIM3_CH4('11')/FT/PC9
- new net N$42: U2U.PA6/SPI1_MISO('0')/TIM8_BKIN/ADC12_IN6/TIM3_CH1('00')/TIM1_BKIN('01')
- new net SRAM_CS1: IC2IC.!CS, U1BANK0.IOT_222
- new net SRAM_CS2: IC3IC.!CS, U1BANK0.IOT_206
- net ADC3: now also U2U.ADC12_IN15/PC5; no longer U2U.ADC123_IN11/PC1
- net ADC4: now also U2U.ADC12_IN14/PC4; no longer U2U.ADC123_IN12/PC2
- net ADC5: now also U2U.PA3/USART2_RX('0')/TIM5_CH4/ADC123_IN3/TIM2_CH4('00'OR'01'); no longer U2U.ADC123_IN10/PC0
- net ADC6: now also U2U.PA7/SPI1_MOSI('0')/TIM8_CH1N/ADC12_IN7/TIM3_CH2('00')/TIM1_CH1N('01'); no longer U2U.ADC12_IN14/PC4
- net IO_OE: now also U1BANK0.IOT_177; no longer U1BANK0.IOT_206
- net MCU_INT0: now also U1BANK0.GBIN0/IOT_198, U2U.UART4_RX/USART3_RX('01')/FT/PC11; no longer U1BANK2.GBIN4/IOB_82
- net MCU_INT1: now also U1BANK0.GBIN1/IOT_197, U2U.UART4_TX/USART3_TX('01')/FT/PC10; no longer U1BANK2.GBIN5/IOB_81
- net N$30: now also U2U.ADC123_IN10/PC0; no longer U2U.PA3/USART2_RX('0')/TIM5_CH4/ADC123_IN3/TIM2_CH4('00'OR'01')
- net N$34: now also U2U.PA5/SPI1_SCK('0')/ADC12_IN5; no longer U2U.PA4/SPI1_NSS('0')/USART2_CK('0')/ADC12_IN4
- net N$35: now also U2U.ADC123_IN11/PC1; no longer U2U.ADC12_IN15/PC5
Other:
- note added: "SRAM_1"
- note added: "SRAM_2"
Changed lines of the file:
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@@
 <text x="-177.8" y="500.38" size="1.778" layer="94">STM32 power rail</text>
 <text x="-256.54" y="495.3" size="2.54" layer="94" ratio="10" align="center">INTERNAL 1.2V VREG</text>
+<text x="55.88" y="563.88" size="1.778" layer="91" rot="R90">SRAM_1</text>
+<text x="55.88" y="535.94" size="1.778" layer="91" rot="R90">SRAM_2</text>
 </plain>
 <instances>
@@
 </segment>
 <segment>
-<label x="-139.7" y="144.78" size="1.778" layer="95" align="center-left"/>
-<pinref part="U2" gate="U" pin="ADC123_IN11/PC1"/>
-<wire x1="-142.24" y1="144.78" x2="-139.7" y2="144.78" width="0.1524" layer="91"/>
+<pinref part="U2" gate="U" pin="ADC12_IN15/PC5"/>
+<wire x1="-142.24" y1="134.62" x2="-139.7" y2="134.62" width="0.1524" layer="91"/>
+<label x="-139.7" y="134.62" size="1.778" layer="95"/>
 </segment>
 </net>
@@
 </segment>
 <segment>
-<label x="-139.7" y="142.24" size="1.778" layer="95" align="center-left"/>
-<pinref part="U2" gate="U" pin="ADC123_IN12/PC2"/>
-<wire x1="-142.24" y1="142.24" x2="-139.7" y2="142.24" width="0.1524" layer="91"/>
+<label x="-139.7" y="137.16" size="1.778" layer="95" align="center-left"/>
+<pinref part="U2" gate="U" pin="ADC12_IN14/PC4"/>
+<wire x1="-142.24" y1="137.16" x2="-139.7" y2="137.16" width="0.1524" layer="91"/>
 </segment>
 </net>
@@
 </segment>
 <segment>
-<label x="-139.7" y="147.32" size="1.778" layer="95" align="center-left"/>
-<pinref part="U2" gate="U" pin="ADC123_IN10/PC0"/>
-<wire x1="-142.24" y1="147.32" x2="-139.7" y2="147.32" width="0.1524" layer="91"/>
+<pinref part="U2" gate="U" pin="PA3/USART2_RX('0')/TIM5_CH4/ADC123_IN3/TIM2_CH4('00'OR'01')"/>
+<wire x1="-248.92" y1="182.88" x2="-251.46" y2="182.88" width="0.1524" layer="91"/>
+<label x="-256.54" y="182.88" size="1.778" layer="95"/>
 </segment>
 </net>
@@
 </segment>
 </net>
-<net name="SRAM_CS" class="0">
-<segment>
-<wire x1="78.74" y1="558.8" x2="81.28" y2="558.8" width="0.1524" layer="91"/>
-<wire x1="78.74" y1="530.86" x2="81.28" y2="530.86" width="0.1524" layer="91"/>
-<wire x1="81.28" y1="530.86" x2="86.36" y2="530.86" width="0.1524" layer="91"/>
-<wire x1="81.28" y1="558.8" x2="81.28" y2="530.86" width="0.1524" layer="91"/>
-<junction x="81.28" y="530.86"/>
-<label x="86.36" y="530.86" size="1.778" layer="95" rot="MR0" align="center-right"/>
-<pinref part="IC2" gate="IC" pin="!CS"/>
-<pinref part="IC3" gate="IC" pin="!CS"/>
-</segment>
-<segment>
-<pinref part="U1" gate="BANK0" pin="IOT_222"/>
-<wire x1="-2.54" y1="482.6" x2="0" y2="482.6" width="0.1524" layer="91"/>
-<label x="0" y="482.6" size="1.778" layer="95"/>
-</segment>
-<segment>
-<pinref part="U2" gate="U" pin="PA15/FT/JTDI/SPI3_NSS('0')/TIM2_CH1_ETR('11')/SPI1_NSS('1')"/>
-<wire x1="-248.92" y1="152.4" x2="-251.46" y2="152.4" width="0.1524" layer="91"/>
-<label x="-261.62" y="152.4" size="1.778" layer="95"/>
-</segment>
-</net>
 <net name="IO_OE" class="0">
 <segment>
@@
 </segment>
 <segment>
-<pinref part="U1" gate="BANK0" pin="IOT_206"/>
-<wire x1="-2.54" y1="457.2" x2="0" y2="457.2" width="0.1524" layer="91"/>
-<label x="0" y="457.2" size="1.778" layer="95"/>
+<pinref part="U1" gate="BANK0" pin="IOT_177"/>
+<wire x1="-38.1" y1="436.88" x2="-40.64" y2="436.88" width="0.1524" layer="91"/>
+<label x="-48.26" y="436.88" size="1.778" layer="95"/>
 </segment>
 </net>
@@
 </segment>
 <segment>
-<label x="-139.7" y="137.16" size="1.778" layer="95" align="center-left"/>
-<pinref part="U2" gate="U" pin="ADC12_IN14/PC4"/>
-<wire x1="-142.24" y1="137.16" x2="-139.7" y2="137.16" width="0.1524" layer="91"/>
+<pinref part="U2" gate="U" pin="PA7/SPI1_MOSI('0')/TIM8_CH1N/ADC12_IN7/TIM3_CH2('00')/TIM1_CH1N('01')"/>
+<wire x1="-248.92" y1="172.72" x2="-251.46" y2="172.72" width="0.1524" layer="91"/>
+<label x="-259.08" y="172.72" size="1.778" layer="95"/>
 </segment>
 </net>
@@
 </segment>
 </net>
-<net name="N$24" class="0">
+<net name="MCU_INT0" class="0">
 <segment>
 <pinref part="U1" gate="BANK0" pin="GBIN0/IOT_198"/>
 <wire x1="-2.54" y1="454.66" x2="0" y2="454.66" width="0.1524" layer="91"/>
+<label x="0" y="454.66" size="1.778" layer="95"/>
 </segment>
-</net>
-<net name="N$25" class="0">
 <segment>
-<pinref part="U1" gate="BANK0" pin="GBIN1/IOT_197"/>
-<wire x1="-2.54" y1="452.12" x2="0" y2="452.12" width="0.1524" layer="91"/>
+<pinref part="U2" gate="U" pin="UART4_RX/USART3_RX('01')/FT/PC11"/>
+<wire x1="-142.24" y1="119.38" x2="-139.7" y2="119.38" width="0.1524" layer="91"/>
+<label x="-139.7" y="119.38" size="1.778" layer="95"/>
 </segment>
 </net>
-<net name="MCU_INT0" class="0">
+<net name="MCU_INT1" class="0">
 <segment>
-<pinref part="U1" gate="BANK2" pin="GBIN4/IOB_82"/>
-<wire x1="78.74" y1="350.52" x2="81.28" y2="350.52" width="0.1524" layer="91"/>
-<label x="81.28" y="350.52" size="1.778" layer="95"/>
+<pinref part="U1" gate="BANK0" pin="GBIN1/IOT_197"/>
+<wire x1="-2.54" y1="452.12" x2="0" y2="452.12" width="0.1524" layer="91"/>
+<label x="0" y="452.12" size="1.778" layer="95"/>
 </segment>
-</net>
-<net name="MCU_INT1" class="0">
 <segment>
-<pinref part="U1" gate="BANK2" pin="GBIN5/IOB_81"/>
-<wire x1="78.74" y1="347.98" x2="81.28" y2="347.98" width="0.1524" layer="91"/>
-<label x="81.28" y="347.98" size="1.778" layer="95"/>
+<pinref part="U2" gate="U" pin="UART4_TX/USART3_TX('01')/FT/PC10"/>
+<wire x1="-142.24" y1="121.92" x2="-139.7" y2="121.92" width="0.1524" layer="91"/>
+<label x="-139.7" y="121.92" size="1.778" layer="95"/>
 </segment>
 </net>
@@
 </segment>
 </net>
-<net name="N$23" class="0">
-<segment>
-<pinref part="U1" gate="BANK0" pin="IOT_177"/>
-<wire x1="-38.1" y1="436.88" x2="-40.64" y2="436.88" width="0.1524" layer="91"/>
-</segment>
-</net>
 <net name="N$11" class="0">
 <segment>
@@
 </segment>
 </net>
-<net name="N$30" class="0">
-<segment>
-<pinref part="U2" gate="U" pin="PA3/USART2_RX('0')/TIM5_CH4/ADC123_IN3/TIM2_CH4('00'OR'01')"/>
-<wire x1="-248.92" y1="182.88" x2="-251.46" y2="182.88" width="0.1524" layer="91"/>
-</segment>
-</net>
 <net name="N$10" class="0">
 <segment>
@@
 </segment>
 </net>
-<net name="N$34" class="0">
-<segment>
-<pinref part="U2" gate="U" pin="PA4/SPI1_NSS('0')/USART2_CK('0')/ADC12_IN4"/>
-<wire x1="-248.92" y1="180.34" x2="-251.46" y2="180.34" width="0.1524" layer="91"/>
-</segment>
-</net>
-<net name="N$35" class="0">
-<segment>
-<pinref part="U2" gate="U" pin="ADC12_IN15/PC5"/>
-<wire x1="-142.24" y1="134.62" x2="-139.7" y2="134.62" width="0.1524" layer="91"/>
-</segment>
-</net>
 <net name="N$36" class="0">
 <segment>
@@
 </segment>
 </net>
+<net name="N$30" class="0">
+<segment>
+<pinref part="U2" gate="U" pin="ADC123_IN10/PC0"/>
+<wire x1="-142.24" y1="147.32" x2="-139.7" y2="147.32" width="0.1524" layer="91"/>
+</segment>
+</net>
+<net name="N$34" class="0">
+<segment>
+<pinref part="U2" gate="U" pin="PA5/SPI1_SCK('0')/ADC12_IN5"/>
+<wire x1="-248.92" y1="177.8" x2="-251.46" y2="177.8" width="0.1524" layer="91"/>
+</segment>
+</net>
+<net name="N$42" class="0">
+<segment>
+<pinref part="U2" gate="U" pin="PA6/SPI1_MISO('0')/TIM8_BKIN/ADC12_IN6/TIM3_CH1('00')/TIM1_BKIN('01')"/>
+<wire x1="-248.92" y1="175.26" x2="-251.46" y2="175.26" width="0.1524" layer="91"/>
+</segment>
+</net>
+<net name="N$35" class="0">
+<segment>
+<pinref part="U2" gate="U" pin="ADC123_IN11/PC1"/>
+<wire x1="-142.24" y1="144.78" x2="-139.7" y2="144.78" width="0.1524" layer="91"/>
+</segment>
+</net>
+<net name="SRAM_CS1" class="0">
+<segment>
+<wire x1="78.74" y1="558.8" x2="81.28" y2="558.8" width="0.1524" layer="91"/>
+<pinref part="IC2" gate="IC" pin="!CS"/>
+<wire x1="81.28" y1="558.8" x2="86.36" y2="558.8" width="0.1524" layer="91"/>
+<label x="86.36" y="558.8" size="1.778" layer="95"/>
+</segment>
+<segment>
+<pinref part="U1" gate="BANK0" pin="IOT_222"/>
+<wire x1="-2.54" y1="482.6" x2="0" y2="482.6" width="0.1524" layer="91"/>
+<label x="0" y="482.6" size="1.778" layer="95"/>
+</segment>
+</net>
+<net name="SRAM_CS2" class="0">
+<segment>
+<wire x1="78.74" y1="530.86" x2="81.28" y2="530.86" width="0.1524" layer="91"/>
+<wire x1="81.28" y1="530.86" x2="86.36" y2="530.86" width="0.1524" layer="91"/>
+<label x="86.36" y="530.86" size="1.778" layer="95" rot="MR0" align="center-right"/>
+<pinref part="IC3" gate="IC" pin="!CS"/>
+</segment>
+<segment>
+<pinref part="U1" gate="BANK0" pin="IOT_206"/>
+<wire x1="-2.54" y1="457.2" x2="0" y2="457.2" width="0.1524" layer="91"/>
+<label x="0" y="457.2" size="1.778" layer="95"/>
+</segment>
+</net>
+<net name="N$41" class="0">
+<segment>
+<pinref part="U2" gate="U" pin="TIM8_CH4/TIM3_CH4('11')/FT/PC9"/>
+<wire x1="-142.24" y1="124.46" x2="-139.7" y2="124.46" width="0.1524" layer="91"/>
+</segment>
+</net>

Commit message: moved BUFDIR_MOSI from IOR_167 to IOR_111 BUFIO_MOSI from IOR_166 to IOR_110 BUFOD_MOSI from IOR_165 to IOR_119 BUFDIR_CLOCK from 164 to IOR_115 BUFIO_CLOCK from 161 to IOR_114 BUFOD_CLOCK from 160 to IOR_112 BUFDIR_MISO from IOR_152 to IOR_118 BUFIO_MISO from IOR_148 to IOR_117 BUFOD_MISO from IOR_147 to IOR_116 BUFDIR_AUX from IOR_144 to IOR_167 BUFIO_AUX from IOR_141 to IOR_166 BUFOD_AUX from IOR_140 to IOR_165 BUFDIR_CS from IOR_139 to IOR_164 BUFIO_CS from IOR_138 to IOR_161 BUFOD_CS from IOR_137 to IOR_160 change pcb size from 85x56 to 100x50 named all VCC net to 3V3
Parts:
- removed PCB2: PCB_DP_RECTANGLE-85X56, dp_blank_pcb:PCB_DP_RECTANGLE-85X56
- added PCB1: PCB_DP_RECTANGLE-50X100, dp_blank_pcb:PCB_DP_RECTANGLE-50X100
Connections:
- net 3V3: now also IC10P.VCC, IC11.VCCA, IC12P.VCC, IC13.VCCA, IC14P.VCC, IC15.VCCA, IC16P.VCC, IC17.VCCA, IC8P.VCC, IC9.VCCA, R22.2, R25.2, R28.2, R31.2, R34.2
- net BUFDIR_AUX: now also U1BANK1.IOR_167; no longer U1BANK1.IOR_144
- net BUFDIR_CLOCK: now also U1BANK1.IOR_115; no longer U1BANK1.IOR_164
- net BUFDIR_CS: now also U1BANK1.IOR_164; no longer U1BANK1.IOR_139
- net BUFDIR_MISO: now also U1BANK1.IOR_118; no longer U1BANK1.IOR_152
- net BUFDIR_MOSI: now also U1BANK1.IOR_111; no longer U1BANK1.IOR_167
- net BUFIO_AUX: now also U1BANK1.IOR_166; no longer U1BANK1.GBIN2/IOR_141
- net BUFIO_CLOCK: now also U1BANK1.IOR_114; no longer U1BANK1.IOR_161
- net BUFIO_CS: now also U1BANK1.IOR_161; no longer U1BANK1.IOR_138
- net BUFIO_MISO: now also U1BANK1.IOR_117; no longer U1BANK1.IOR_148
- net BUFIO_MOSI: now also U1BANK1.IOR_110; no longer U1BANK1.IOR_166
- net BUFOD_AUX: now also U1BANK1.IOR_165; no longer U1BANK1.GBIN3/IOR_140
- net BUFOD_CLOCK: now also U1BANK1.IOR_112; no longer U1BANK1.IOR_160
- net BUFOD_CS: now also U1BANK1.IOR_160; no longer U1BANK1.IOR_137
- net BUFOD_MISO: now also U1BANK1.IOR_116; no longer U1BANK1.IOR_147
- net BUFOD_MOSI: now also U1BANK1.IOR_109; no longer U1BANK1.IOR_165
- net VCC: no longer IC10P.VCC, IC11.VCCA, IC12P.VCC, IC13.VCCA, IC14P.VCC, IC15.VCCA, IC16P.VCC, IC17.VCCA, IC8P.VCC, IC9.VCCA, R22.2, R25.2, R28.2, R31.2, R34.2
Other:
- moved on the sheet: C12, C32, IC10, IC10P, IC11, IC12, IC12P, IC13, IC14, IC14P, IC15, IC16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
