File: hardware/scratch/BusPirate-ultra.v1.0a.brd (EAGLE design)
At the start: 100 x 50 mm, 136 parts, among them IC1 IC_MEM_23LC1024, IC10 IC_BUFF_SN74LVC1T45DBV, IC11 IC_BUFF_SN74LVC1T45DBV, IC12 74LVC1G07DBV, IC13 IC_BUFF_SN74LVC1T45DBV, IC14 IC_BL1551, IC15 IC_BL1551, IC16 74HCT4066PW, IC2 IC_MEM_23LC1024, IC3 IC_74AC573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

Commit message: increment version to Bus Pirate Ultra v1.0a, removed previous BusPirate-ng.v4.0 files flash CS pin wired to GND fix ARM and FPGA chip pin 1 indicator fix bl1331 pin 1
Connections:
- net 3V3: now also U1.1
- net GND: no longer U1.1
Routing:
- net 3V3: track 512.4 -> 513.8 mm
Other:
- board text added: "Bus Pirate Ultra v1.0a"
- board text removed: "Bus Pirate Ultra v1.0"
Changed lines of the file:
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@@
 <text x="80" y="48.8" size="1.524" layer="21" font="vector" ratio="15" rot="R180" align="center">VREG</text>
 <text x="-3.7338" y="26.8704" size="1.27" layer="49" ratio="10" rot="SR270">USB</text>
-<text x="18.1483" y="25.0842" size="2.4384" layer="22" ratio="12" rot="SMR270" align="center">Bus Pirate Ultra v1.0</text>
+<text x="18.1483" y="25.0842" size="2.4384" layer="22" ratio="12" rot="SMR270" align="center">Bus Pirate Ultra v1.0a</text>
 <text x="20" y="48.8" size="1.524" layer="22" font="vector" ratio="15" rot="MR180" align="center">PWR</text>
 <text x="60" y="48.8" size="1.524" layer="22" font="vector" ratio="15" rot="MR180" align="center">MODE</text>
@@
 <text x="88.9" y="28.575" size="1.016" layer="22" font="vector" ratio="15" rot="MR0" align="center-right">VPU</text>
 <text x="88.9" y="15.875" size="1.016" layer="22" font="vector" ratio="15" rot="MR0" align="center-right">CLK</text>
-<text x="50" y="1.27" size="1.9304" layer="21" ratio="12" rot="R180" align="center">Bus Pirate Ultra v1.0</text>
+<text x="50" y="1.27" size="1.9304" layer="21" ratio="12" rot="R180" align="center">Bus Pirate Ultra v1.0a</text>
 <text x="2.54" y="13.97" size="1.27" layer="21" font="vector" ratio="12" rot="R90" align="center">MAY 2019</text>
 <text x="33.02" y="45.085" size="0.9144" layer="25" font="vector" ratio="12" rot="SR90" align="center-right">SW-
@@
 <via x="19.812" y="19.4564" extent="1-16" drill="0.508"/>
 <contactref element="U1" pad="4"/>
-<contactref element="U1" pad="1"/>
 <contactref element="C2" pad="1"/>
 </signal>
@@
 <wire x1="22.225" y1="45.46693125" x2="22.92866875" y2="46.1706" width="0.254" layer="1"/>
 <wire x1="24.96873125" y1="46.1706" x2="25.545" y2="46.74686875" width="0.254" layer="1"/>
-<wire x1="22.92866875" y1="46.1706" x2="24.96873125" y2="46.1706" width="0.254" layer="1"/>
+<wire x1="22.92866875" y1="46.1706" x2="24.765" y2="46.1706" width="0.254" layer="1"/>
+<wire x1="24.765" y1="46.1706" x2="24.96873125" y2="46.1706" width="0.254" layer="1"/>
 <wire x1="25.545" y1="46.74686875" x2="25.545" y2="47" width="0.254" layer="1"/>
 <wire x1="22.225" y1="44.6878" x2="22.225" y2="45.46693125" width="0.254" layer="1"/>
@@
 <wire x1="26.67" y1="41.87" x2="26.71" y2="41.91" width="0.4064" layer="1"/>
 <wire x1="26.71" y1="41.91" x2="27.94" y2="41.91" width="0.4064" layer="1"/>
+<contactref element="U1" pad="1"/>
+<wire x1="24.765" y1="44.6878" x2="24.765" y2="46.1706" width="0.254" layer="1"/>
 </signal>
 <signal name="N$7">
