File: hardware/scratch/BusPirate-ultra.v1.0b.sch (EAGLE design)
At the start: 174 parts, among them IC1 23LC1024, IC10 SN74LVC1T45DBV, IC11 SN74LVC1T45DBV, IC12 74LVC1G07DBV, IC13 SN74LVC1T45DBV, IC17 74LVC1G07DBV, IC18 SN74LVC1T45DBV, IC19 74LVC1G07DBV, IC2 23LC1024, IC20 SN74LVC1T45DBV, IC21 74LVC1G07DBV, IC22 SN74LVC1T45DBV, IC23 MCP1824_ADJ, IC24 74HCT4051, IC3 74AC573, IC4 74LVC1G07DBV, IC5 74LVC1G07DBV, IC6 74LVC1G07DBV, IC7 74LVC1G07DBV, IC8 SN74LVC1T45DBV, IC9 SN74LVC1T45DBV, J2 CON_HEADER_1X04, J4 CON_HEADER_1X10-RIGHT_ANGLED_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, Q1 DMMT3906W, U1 W25X40CL, U2 STM32F103ZX, U3 ICE40HX4K, U4 MCP6001, U5 MCP4442, U6 MCP4442, U7 MCP6001

Commit message: place 0R resistor on the feedback of vreg DAC buffer and placed an rc filter on the input. replace with 10uF cap on the adj vreg chip input. change buffer chip with an SC-70 packages and 0402 caps and resitors
Parts:
- added R48: (no value), dp_devices.v6:RESISTOR-0603
- added R53: 0R, dp_devices.v6:RESISTOR-0603
- C40, C41, C42, C43, C46, C47, C48, C49: device rcl:C-EUC0603 -> resistor:C-EUC0402
- C63: value 0.1uF -> 10uF
- IC10, IC11, IC13, IC18, IC20, IC22, IC9: device dp_devices.v6:IC_BUFF_SN74LVC1T45DBV -> dp_devices.v6:IC_BUFF_SN74LVC1T45DBV-SC-70-6
- IC12, IC17, IC19, IC21, IC5, IC6, IC7: device 74xx-little-de:74LVC1G07DBV -> dp_devices.v6:IC_BUFF_74LVC1G07
- R19, R24, R28: device rcl:R-EU_R0402 -> resistor:R-EU_R0402
- R20, R21, R22, R23, R25, R26, R27, R29, R30, R31, R32, R33, R40: device rcl:R-EU_R0603 -> resistor:R-EU_R0402
Connections:
- new net N$15: R53.1, U4.-
- new net N$31: C53.1, R48.2, U4.+
- net 3V3: now also IC12P.V+, IC17P.V+, IC19P.V+, IC21P.V+, IC5P.V+, IC6P.V+, IC7P.V+; no longer IC12P.VCC, IC17P.VCC, IC19P.VCC, IC21P.VCC, IC5P.VCC, IC6P.VCC, IC7P.VCC
- net BPIO1: now also IC5G.O; no longer IC5A.O
- net BPIO2: now also IC6G.O; no longer IC6A.O
- net BPIO3: now also IC12G.O; no longer IC12A.O
- net BPIO4: now also IC7G.O; no longer IC7A.O
- net BPIO5: now also IC17G.O; no longer IC17A.O
- net BPIO6: now also IC19G.O; no longer IC19A.O
- net BPIO7: now also IC21G.O; no longer IC21A.O
- net BUFOD1: now also IC5G.I; no longer IC5A.I
- net BUFOD2: now also IC6G.I; no longer IC6A.I
- net BUFOD3: now also IC12G.I; no longer IC12A.I
- net BUFOD4: now also IC7G.I; no longer IC7A.I
- net BUFOD5: now also IC17G.I; no longer IC17A.I
- net BUFOD6: now also IC19G.I; no longer IC19A.I
- net BUFOD7: now also IC21G.I; no longer IC21A.I
- net N$25: now also R53.2; no longer U4.-
- net VREG_DAC: now also R48.1; no longer C53.1, U4.+
Other:
- moved on the sheet: C53, C61, C63, C64, IC12P, IC17P, IC19P, IC21P, IC23, IC4P, IC5P, IC6P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
