File: hardware/scratch/BusPirate-ultra.v1.0b.sch (EAGLE design)
At the start: 166 parts, among them IC1 23LC1024, IC10 SN74LVC1T45DBV, IC11 SN74LVC1T45DBV, IC12 74LVC1G07DBV, IC13 SN74LVC1T45DBV, IC17 74LVC1G07DBV, IC18 SN74LVC1T45DBV, IC19 74LVC1G07DBV, IC2 23LC1024, IC20 SN74LVC1T45DBV, IC21 74LVC1G07DBV, IC22 SN74LVC1T45DBV, IC23 MCP1824_ADJ, IC24 74HCT4051, IC4 74LVC1G07DBV, IC5 74LVC1G07DBV, IC6 74LVC1G07DBV, IC7 74LVC1G07DBV, IC8 SN74LVC1T45DBV, IC9 SN74LVC1T45DBV, J1 CON_MOLEX_MALE_SMT_SH_1.25, J2 CON_HEADER_1X04, J4 CON_HEADER_1X10-RIGHT_ANGLED_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, Q1 DMMT3906W, U1 W25X40CL, U2 STM32F103ZX, U3 ICE40HX4K, U4 MCP6001, U5 74LVC245A, U7 MCP6001, U8 74HCT4066PW, U9 74HCT4066PW

Commit message: move pins arrangement on diplay connector Display PWM pin is now on pin 46/PB0 move MCU_AUX11 from PC5 to PF14 move MCU_AUX10 from PB0 to PG1 tried to move ADX mux near the 245 chip
Connections:
- removed net ADC6: U2U.ADC12_IN14/PC4
- removed net N$62: J1.8
- new net DISPLAY_PWM: J1.3, U2U.ADC12_IN8/TIM3_CH3('00'OR'10')/TIM8_CH2N/TIM1_CH2N('01')/PB0
- new net N$48: U2U.ADC12_IN15/PC5
- net 3V3: now also J1.7; no longer J1.6
- net DISPLAY_CS: now also J1.1, U2U.FSMC_A6/FT/PF12; no longer J1.4
- net DISPLAY_D/P: now also J1.2, U2U.FSMC_NIOS16/FT/PF11; no longer J1.5
- net DISPLAY_SPI_CLOCK: now also J1.6; no longer J1.1
- net DISPLAY_SPI_MISO: now also J1.5; no longer J1.2
- net DISPLAY_SPI_MOSI: now also J1.4; no longer J1.3
- net GND: now also J1.8; no longer J1.7
- net MCU_AUX10: now also U2U.PG1/FT/FSMC_A11; no longer U2U.ADC12_IN8/TIM3_CH3('00'OR'10')/TIM8_CH2N/TIM1_CH2N('01')/PB0
- net MCU_AUX11: now also U2U.FSMC_A8/FT/PF14; no longer U2U.ADC12_IN15/PC5
- net N$28: now also U2U.PD11/FT/FSMC_A16/USART3_CTS('11'); no longer U2U.PA0/WKUP/USART2_CTS('0')/ADC123_IN0/TIM2_CH1_ETR/TIM5_CH1/TIM8_ETR
- net VREGEN: now also U2U.PE5/FT/FSMC_A21; no longer U2U.FSMC_A8/FT/PF14
Changed lines of the file:
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@@
 <instance part="U5" gate="SUPPLY" x="505.46" y="330.2"/>
 <instance part="J1" gate="J" x="711.2" y="55.88"/>
-<instance part="GND69" gate="G$1" x="701.04" y="50.8" smashed="yes"/>
+<instance part="GND69" gate="G$1" x="701.04" y="48.26" smashed="yes"/>
 </instances>
 <busses>
@@
 </segment>
 <segment>
-<pinref part="J1" gate="J" pin="7"/>
-<wire x1="711.2" y1="53.34" x2="706.12" y2="53.34" width="0.1524" layer="91"/>
+<pinref part="J1" gate="J" pin="8"/>
 <pinref part="GND69" gate="G$1" pin="GND"/>
-<wire x1="706.12" y1="53.34" x2="701.04" y2="53.34" width="0.1524" layer="91"/>
+<wire x1="711.2" y1="50.8" x2="701.04" y2="50.8" width="0.1524" layer="91"/>
 </segment>
 </net>
@@
 </segment>
 <segment>
-<pinref part="J1" gate="J" pin="6"/>
-<wire x1="711.2" y1="55.88" x2="706.12" y2="55.88" width="0.1524" layer="91"/>
-<label x="706.12" y="55.88" size="1.778" layer="95" align="center-right"/>
+<pinref part="J1" gate="J" pin="7"/>
+<wire x1="711.2" y1="53.34" x2="706.12" y2="53.34" width="0.1524" layer="91"/>
+<label x="706.12" y="53.34" size="1.778" layer="95" align="center-right"/>
 </segment>
 </net>
@@
 </segment>
 <segment>
-<label x="147.32" y="307.34" size="1.778" layer="95" align="center-left"/>
-<pinref part="U2" gate="U" pin="FSMC_A8/FT/PF14"/>
-<wire x1="147.32" y1="307.34" x2="144.78" y2="307.34" width="0.1524" layer="91"/>
-</segment>
-<segment>
 <pinref part="IC23" gate="IC" pin="!SHDN"/>
 <wire x1="335.28" y1="322.58" x2="330.2" y2="322.58" width="0.1524" layer="91"/>
@@
 <label x="325.12" y="322.58" size="1.778" layer="95" align="center-right"/>
 </segment>
+<segment>
+<pinref part="U2" gate="U" pin="PE5/FT/FSMC_A21"/>
+<wire x1="38.1" y1="330.2" x2="35.56" y2="330.2" width="0.1524" layer="91"/>
+<label x="35.56" y="330.2" size="1.778" layer="95" align="center-right"/>
+</segment>
 </net>
 <net name="N$18" class="0">
@@
 </segment>
 </net>
-<net name="ADC6" class="0">
-<segment>
-<pinref part="U2" gate="U" pin="ADC12_IN14/PC4"/>
-<wire x1="144.78" y1="375.92" x2="147.32" y2="375.92" width="0.1524" layer="91"/>
-<label x="147.32" y="375.92" size="1.778" layer="95" align="center-left"/>
-</segment>
-</net>
 <net name="UART_RX" class="0">
 <segment>
@@
 </segment>
 </net>
-<net name="N$28" class="0">
-<segment>
-<pinref part="U2" gate="U" pin="PA0/WKUP/USART2_CTS('0')/ADC123_IN0/TIM2_CH1_ETR/TIM5_CH1/TIM8_ETR"/>
-<wire x1="38.1" y1="429.26" x2="35.56" y2="429.26" width="0.1524" layer="91"/>
-</segment>
-</net>
 <net name="N$36" class="0">
 <segment>
@@
 </segment>
 <segment>
-<pinref part="U2" gate="U" pin="ADC12_IN8/TIM3_CH3('00'OR'10')/TIM8_CH2N/TIM1_CH2N('01')/PB0"/>
-<wire x1="144.78" y1="299.72" x2="147.32" y2="299.72" width="0.1524" layer="91"/>
-<label x="147.32" y="299.72" size="1.778" layer="95" align="center-left"/>
+<pinref part="U2" gate="U" pin="PG1/FT/FSMC_A11"/>
+<wire x1="38.1" y1="297.18" x2="35.56" y2="297.18" width="0.1524" layer="91"/>
+<label x="35.56" y="297.18" size="1.778" layer="95" align="center-right"/>
 </segment>
 </net>
@@
 </segment>
 <segment>
-<pinref part="U2" gate="U" pin="ADC12_IN15/PC5"/>
-<wire x1="144.78" y1="373.38" x2="147.32" y2="373.38" width="0.1524" layer="91"/>
-<label x="147.32" y="373.38" size="1.778" layer="95" align="center-left"/>
+<pinref part="U2" gate="U" pin="FSMC_A8/FT/PF14"/>
+<wire x1="144.78" y1="307.34" x2="147.32" y2="307.34" width="0.1524" layer="91"/>
+<label x="147.32" y="307.34" size="1.778" layer="95" align="center-left"/>
 </segment>
 </net>
@@
 </segment>
 <segment>
-<pinref part="J1" gate="J" pin="1"/>
-<wire x1="711.2" y1="68.58" x2="706.12" y2="68.58" width="0.1524" layer="91"/>
-<label x="706.12" y="68.58" size="1.778" layer="95" align="center-right"/>
+<pinref part="J1" gate="J" pin="6"/>
+<wire x1="711.2" y1="55.88" x2="706.12" y2="55.88" width="0.1524" layer="91"/>
+<label x="706.12" y="55.88" size="1.778" layer="95" align="center-right"/>
 </segment>
 </net>
@@
 </segment>
 <segment>
-<pinref part="J1" gate="J" pin="3"/>
-<wire x1="711.2" y1="63.5" x2="706.12" y2="63.5" width="0.1524" layer="91"/>
-<label x="706.12" y="63.5" size="1.778" layer="95" align="center-right"/>
+<pinref part="J1" gate="J" pin="4"/>
+<wire x1="711.2" y1="60.96" x2="706.12" y2="60.96" width="0.1524" layer="91"/>
+<label x="706.12" y="60.96" size="1.778" layer="95" align="center-right"/>
 </segment>
 </net>
@@
 </segment>
 <segment>
-<pinref part="J1" gate="J" pin="2"/>
-<wire x1="711.2" y1="66.04" x2="706.12" y2="66.04" width="0.1524" layer="91"/>
-<label x="706.12" y="66.04" size="1.778" layer="95" align="center-right"/>
+<pinref part="J1" gate="J" pin="5"/>
+<wire x1="711.2" y1="58.42" x2="706.12" y2="58.42" width="0.1524" layer="91"/>
+<label x="706.12" y="58.42" size="1.778" layer="95" align="center-right"/>
 </segment>
 </net>
@@
 <net name="DISPLAY_CS" class="0">
 <segment>
-<pinref part="J1" gate="J" pin="4"/>
-<wire x1="711.2" y1="60.96" x2="706.12" y2="60.96" width="0.1524" layer="91"/>
-<label x="706.12" y="60.96" size="1.778" layer="95" align="center-right"/>
+<pinref part="J1" gate="J" pin="1"/>
+<wire x1="711.2" y1="68.58" x2="706.12" y2="68.58" width="0.1524" layer="91"/>
+<label x="706.12" y="68.58" size="1.778" layer="95" align="center-right"/>
+</segment>
+<segment>
+<pinref part="U2" gate="U" pin="FSMC_A6/FT/PF12"/>
+<wire x1="144.78" y1="312.42" x2="147.32" y2="312.42" width="0.1524" layer="91"/>
+<label x="147.32" y="312.42" size="1.778" layer="95" align="center-left"/>
 </segment>
 </net>
 <net name="DISPLAY_D/P" class="0">
 <segment>
-<pinref part="J1" gate="J" pin="5"/>
-<wire x1="711.2" y1="58.42" x2="706.12" y2="58.42" width="0.1524" layer="91"/>
-<label x="706.12" y="58.42" size="1.778" layer="95" align="center-right"/>
+<pinref part="J1" gate="J" pin="2"/>
+<wire x1="711.2" y1="66.04" x2="706.12" y2="66.04" width="0.1524" layer="91"/>
+<label x="706.12" y="66.04" size="1.778" layer="95" align="center-right"/>
 </segment>
-</net>
-<net name="N$62" class="0">
 <segment>
-<pinref part="J1" gate="J" pin="8"/>
-<wire x1="711.2" y1="50.8" x2="706.12" y2="50.8" width="0.1524" layer="91"/>
+<pinref part="U2" gate="U" pin="FSMC_NIOS16/FT/PF11"/>
+<wire x1="144.78" y1="314.96" x2="147.32" y2="314.96" width="0.1524" layer="91"/>
+<label x="147.32" y="314.96" size="1.778" layer="95" align="center-left"/>
 </segment>
 </net>
@@
 </segment>
 </net>
+<net name="DISPLAY_PWM" class="0">
+<segment>
+<pinref part="U2" gate="U" pin="ADC12_IN8/TIM3_CH3('00'OR'10')/TIM8_CH2N/TIM1_CH2N('01')/PB0"/>
+<wire x1="144.78" y1="299.72" x2="147.32" y2="299.72" width="0.1524" layer="91"/>
+<label x="147.32" y="299.72" size="1.778" layer="95"/>
+</segment>
+<segment>
+<pinref part="J1" gate="J" pin="3"/>
+<wire x1="711.2" y1="63.5" x2="706.12" y2="63.5" width="0.1524" layer="91"/>
+<label x="706.12" y="63.5" size="1.778" layer="95" align="center-right"/>
+</segment>
+</net>
+<net name="N$28" class="0">
+<segment>
+<pinref part="U2" gate="U" pin="PD11/FT/FSMC_A16/USART3_CTS('11')"/>
+<wire x1="38.1" y1="358.14" x2="35.56" y2="358.14" width="0.1524" layer="91"/>
+</segment>
+</net>
+<net name="N$48" class="0">
+<segment>
+<pinref part="U2" gate="U" pin="ADC12_IN15/PC5"/>
+<wire x1="144.78" y1="373.38" x2="147.32" y2="373.38" width="0.1524" layer="91"/>
+</segment>
+</net>

Commit message: Details of Changes listed below: wired 2 additional aux pins from MCU pin 44 and 45 to display connector
rewired ADC mux control pins ADC_MUX_S0..S2 and enable from FPGA Bank 2 to bank 1
ADC_MUX_S0 93
ADC_MUX_S1 94
ADC_MUX_S2 95
ADC_MUX_EN 96

moved MCU_AUX5 from FPGA 125 to 130
moved MCU_AUX6 from FPGA 124 to 125
moved MCU_AUX7 from FPGA 119 to 124
moved MCU_AUX8 from FPGA 118 to 122

moved SRAM1 pins of FPGA

moved buffer 1 control FPGA pins from bank 1 to bank 0
BUFDIR1 from 105 to 110
BUFOD1 from 106 to 112
BUFIO1 from 107 to 113

moved buffer 0 pins
BUFIO0 from 104 to 106
BUFOD0 from 102 to 105
BUFDIR0 from 101 to 107

moved buffer 3 pins
BUFIO3 from 99 to 102
BUFOD3 from 98 to 101
BUFDIR3 from 97 to 104

moved buffer 2 pins
BUFIO2 from 96 to 98
BUFOD2 from 95 to 97
BUFDIR2 from 94 to 99

moved buffer 7 pins
BUFIO7 from 63 to 60
BUFOD7 from 62 to 56
BUFDIR7 from 64 to 61

moved buffer 6 control FPGA pins from bank 1 to bank 2
BUFDIR6 from 75 to 64
BUFOD6 from 73 to 62
BUFIO6 from 74 to 63

moved buffer 5 pins
BUFIO5 from 78 to 74
BUFOD5 from 76 to 73
BUFDIR5 from 79 to 75

moved buffer 4 pins
BUFIO4 from 81 to 78
BUFOD4 from 80 to 76
BUFDIR4 from 82 to 79

move FPGA LAT pins, one pin down
LAT0 91
LAT1 90
LAT2 88
LAT3 87
LAT4 85
LAT5 84
LAT6 83
LAT7 82

decoupling caps still placed on the bottom, so far these places them near the appropriate power pins for the FPGA and other chips
Connections:
- removed net N$14: U3BANK0.IOT_190
- removed net N$16: U3BANK0.IOT_181
- removed net N$20: U3BANK0.IOT_179
- removed net N$21: U3BANK0.IOT_206
- removed net N$24: U3BANK0.IOT_168
- removed net N$48: U2U.ADC12_IN15/PC5
- removed net N$63: J1.9
- removed net N$66: J1.10
- new net DISPLAY_AUX1: J1.5, U2U.ADC12_IN14/PC4
- new net DISPLAY_AUX2: J1.4, U2U.ADC12_IN15/PC5
- net 3V3: now also J1.9; no longer J1.7
- net ADC_MUX_EN: now also U3BANK1.IOR_146; no longer U3BANK2.IOB_96
- net ADC_MUX_S0: now also U3BANK1.GBIN3/IOR_140; no longer U3BANK2.IOB_91
- net ADC_MUX_S1: now also U3BANK1.GBIN2/IOR_141; no longer U3BANK2.IOB_94
- net ADC_MUX_S2: now also U3BANK1.IOR_144; no longer U3BANK2.IOB_95
- net BUFDIR0: now also U3BANK1.IOR_167; no longer U3BANK1.IOR_160
- net BUFDIR1: now also U3BANK0.IOT_170; no longer U3BANK1.IOR_165
- net BUFDIR2: now also U3BANK1.IOR_152; no longer U3BANK1.GBIN2/IOR_141
- net BUFDIR3: now also U3BANK1.IOR_164; no longer U3BANK1.IOR_147
- net BUFDIR4: now also U3BANK1.IOR_115; no longer U3BANK1.IOR_118
- net BUFDIR5: now also U3BANK1.IOR_111; no longer U3BANK1.IOR_115
- net BUFDIR6: now also U3BANK2.CBSEL1/IOB_104; no longer U3BANK1.IOR_111
- net BUFDIR7: now also U3BANK2.IOB_96; no longer U3BANK2.CBSEL1/IOB_104
- net BUFIO0: now also U3BANK1.IOR_166; no longer U3BANK1.IOR_164
- net BUFIO1: now also U3BANK0.IOT_169; no longer U3BANK1.IOR_167
- net BUFIO2: now also U3BANK1.IOR_148; no longer U3BANK1.IOR_146
- net BUFIO3: now also U3BANK1.IOR_161; no longer U3BANK1.IOR_152
- net BUFIO4: now also U3BANK1.IOR_114; no longer U3BANK1.IOR_117
- net BUFIO5: now also U3BANK1.IOR_110; no longer U3BANK1.IOR_114
- net BUFIO6: now also U3BANK2.CBSEL0/IOB_103; no longer U3BANK1.IOR_110
- net BUFIO7: now also U3BANK2.IOB_95; no longer U3BANK2.CBSEL0/IOB_103
- net BUFOD0: now also U3BANK1.IOR_165; no longer U3BANK1.IOR_161
- net BUFOD1: now also U3BANK0.IOT_168; no longer U3BANK1.IOR_166
- net BUFOD2: now also U3BANK1.IOR_147; no longer U3BANK1.IOR_144
- net BUFOD3: now also U3BANK1.IOR_160; no longer U3BANK1.IOR_148
- net BUFOD4: now also U3BANK1.IOR_112; no longer U3BANK1.IOR_116
- net BUFOD5: now also U3BANK1.IOR_109; no longer U3BANK1.IOR_112
- net BUFOD6: now also U3BANK2.IOB_102; no longer U3BANK1.IOR_109
- net BUFOD7: now also U3BANK2.IOB_94; no longer U3BANK2.IOB_102
- net DISPLAY_SPI_CLOCK: now also J1.8; no longer J1.6
- net DISPLAY_SPI_MISO: now also J1.7; no longer J1.5
- net DISPLAY_SPI_MOSI: now also J1.6; no longer J1.4
- net GND: now also J1.10; no longer J1.8
- net LAT0: now also U3BANK1.IOR_139; no longer U3BANK1.GBIN3/IOR_140
- net LAT1: now also U3BANK1.IOR_138; no longer U3BANK1.IOR_139
- net LAT2: now also U3BANK1.IOR_137; no longer U3BANK1.IOR_138
- net LAT3: now also U3BANK1.IOR_136; no longer U3BANK1.IOR_137
- net LAT4: now also U3BANK1.IOR_128; no longer U3BANK1.IOR_136
- net LAT5: now also U3BANK1.IOR_120; no longer U3BANK1.IOR_128
- net LAT6: now also U3BANK1.IOR_119; no longer U3BANK1.IOR_120
- net LAT7: now also U3BANK1.IOR_118; no longer U3BANK1.IOR_119
- net MCU_AUX5: now also U3BANK0.IOT_206; no longer U3BANK0.IOT_192
- net MCU_AUX6: now also U3BANK0.IOT_192; no longer U3BANK0.IOT_191
- net MCU_AUX7: now also U3BANK0.IOT_191; no longer U3BANK0.IOT_178
- net MCU_AUX8: now also U3BANK0.IOT_190; no longer U3BANK0.IOT_177
- net SRAM1_CLOCK: now also U3BANK0.IOT_177; no longer U3BANK0.IOT_171
- net SRAM1_CS: now also U3BANK0.IOT_181; no longer U3BANK0.IOT_174
- net SRAM1_SIO0: now also U3BANK0.IOT_173; no longer U3BANK0.IOT_169
- net SRAM1_SIO1: now also U3BANK0.IOT_178; no longer U3BANK0.IOT_172
- net SRAM1_SIO2: now also U3BANK0.IOT_174; no longer U3BANK0.IOT_170
- net SRAM1_SIO3: now also U3BANK0.IOT_179; no longer U3BANK0.IOT_173

Commit message: change to USB-C, move USB_DET pin from pin 3 to 5/PE6, working on voltage regulator part
Parts:
- removed USB1: MINI-B, dp_devices.v6:CON-USB-F-MINI-B
- added U$3: USB-C-12, usbc:USB-C-12
- L1: value 1.5A ferrite bead -> 1.5A
- R1, R2, R3: device dp_devices.v6:RESISTOR-0603 -> rcl:R-EU_R0603
Connections:
- removed net EXVUSB: L1.1, USB1USB.VUSB
- new net N$1: L1.1, U$3.VBUS
- new net N$16: U2U.OSC32_OUT/PC15
- net D+: now also U$3.DP1, U$3.DP2; no longer USB1USB.D+
- net D-: now also U$3.DN1, U$3.DN2; no longer USB1USB.D-
- net GND: now also U$3.CC1, U$3.CC2, U$3.CHASSIS, U$3.GND; no longer USB1BODY.BODY@1, USB1BODY.BODY@2, USB1BODY.BODY@3, USB1BODY.BODY@4, USB1USB.GND
- net USB_DET: now also U2U.PE6/FT/FSMC_A22; no longer U2U.PE4/FT/FSMC_A20
Other:
- moved on the sheet: C1, L1, R11, R12
